File: PCB/hackpad.kicad_pcb (KiCad board)
At the start: 2 copper layers, 43.4 x 81 mm, 5 parts, among them SW1 SW_Push, SW2 SW_Push, SW3 SW_Push, SW4 SW_Push, U1 XIAO-RP2040-DIP

Commit message: new pcb
Parts:
- added D1: SK6812MINI, LED_SMD:LED_SK6812MINI_PLCC4_3.5x3.5mm_P1.75mm, F.Cu at (62.2, 51.5)
- added D3: SK6812MINI, LED_SMD:LED_SK6812MINI_PLCC4_3.5x3.5mm_P1.75mm, F.Cu at (62.2, 61.8)
- added D5: SK6812MINI, LED_SMD:LED_SK6812MINI_PLCC4_3.5x3.5mm_P1.75mm, F.Cu at (62.2, 103.9)
- added D7: SK6812MINI, LED_SMD:LED_SK6812MINI_PLCC4_3.5x3.5mm_P1.75mm, F.Cu at (62.2, 114.1)
Connections:
- U1 pad 5: unconnected-(U1-GPIO6/SDA-Pad5) -> Net-(D1-DIN)
- U1 pad 6: unconnected-(U1-GPIO7/SCL-Pad6) -> Net-(D5-DIN)
Routing:
- net GND: track 131.8 -> 262.7 mm
- net +5V: track 0.00 -> 127.1 mm
- net Net-(D5-DIN): track 0.00 -> 34.5 mm
- net Net-(D1-DIN): track 0.00 -> 24.8 mm
- net Net-(D1-DOUT): track 0.00 -> 15.2 mm
- net Net-(D5-DOUT): track 0.00 -> 14.4 mm
- net Net-(U1-GPIO4/MISO): track 23.9 -> 27.8 mm
Other:
- board text added: "VaultPad v1.0.0"
- board text removed: "PlumPad v1.0.0"
