File: PCB/hackpad.kicad_sch (KiCad schematic)
At the start: 5 parts, among them SW1 SW_Push, SW2 SW_Push, SW3 SW_Push, SW4 SW_Push, U1 XIAO-RP2040-DIP

Commit message: new pcb
Parts:
- added D1, D3, D5, D7: SK6812MINI, LED_SMD:LED_SK6812MINI_PLCC4_3.5x3.5mm_P1.75mm, symbol LED:SK6812MINI
Connections:
- net +5V: now also D1.4 (VDD), D3.4 (VDD), D5.4 (VDD), D7.4 (VDD)
- net GND: now also D1.2 (VSS), D3.2 (VSS), D5.2 (VSS), D7.2 (VSS)
- net at U1.5 (GPIO6/SDA): now also D1.3 (DIN)
- net at U1.6 (GPIO7/SCL): now also D5.3 (DIN)
- new net: D1.1 (DOUT), D3.3 (DIN)
- new net: D5.1 (DOUT), D7.3 (DIN)
